File: Closed Loop Motor Driver CCA/Closed Loop Motor Driver/Closed Loop Motor Driver.kicad_sch (KiCad schematic)
At the start: 11 parts, among them J1 JST 1x4, J2 JST 1X6, J3 HEADER 1x7 socket, J4 Conn_01x03_Pin, J5 Screw_Terminal_01x03, J6 Screw_Terminal_01x02, U1 SC0915, U7 TXB0108DQSR

Commit message: collected unused signals into connectors
Parts:
- added J7: JST 1x4, symbol Connector:Conn_01x04_Pin
- added J8: Conn_02x05_Counter_Clockwise, symbol Connector_Generic:Conn_02x05_Odd_Even
- added SW1: SW_Push, symbol Switch:SW_Push
- U1: value SC0915 -> RPI PICO
Connections:
- net +3.3V: now also J7.1 (Pin_1), J8.1 (Pin_1)
- net GND: now also J7.2 (Pin_2), J8.2 (Pin_2), SW1.1
- net SPI_CAN_ENABLE: now reaches R8.1, U7.6 (OE)
- net SPI_CAN_ENABLE: now also U1.29 (GP22)
- net UNUSED_GP0: now reaches U1.1 (GP0)
- net UNUSED_GP0: now also J8.3 (Pin_3)
- net UNUSED_GP8: now reaches U1.11 (GP8)
- net UNUSED_GP8: now also J8.9 (Pin_9)
- net UNUSED_GP9: now reaches U1.12 (GP9)
- net UNUSED_GP9: now also J8.4 (Pin_4)
- net ENC_QUAD_A: now reaches U1.19 (GP14)
- net ENC_QUAD_A: now also J7.3 (Pin_3)
- net UNUSED_GP1: now reaches U1.2 (GP1)
- net UNUSED_GP1: now also J8.5 (Pin_5)
- net ENC_QUAD_B: now reaches U1.20 (GP15)
- net ENC_QUAD_B: now also J7.4 (Pin_4)
- net SPI_ADC_ENABLE: now reaches U1.27 (GP21)
- net at U1.30 (~{RUN}): now also SW1.2
- net UNUSED_GP26-A: now reaches U1.31 (GP26)
- net UNUSED_GP26-A: now also J8.6 (Pin_6)
- net UNUSED_GP27-A: now reaches U1.32 (GP27)
- net UNUSED_GP27-A: now also J8.8 (Pin_8)
- net UNUSED_GP28-A: now reaches U1.34 (GP28)
- net UNUSED_GP28-A: now also J8.10 (Pin_10)
- net UNUSED_GP3: now reaches U1.5 (GP3)
- net UNUSED_GP3: now also J8.7 (Pin_7)
- no-connect marks 0 -> 17
Other:
- sheet Analog ports: added ADC_SPI_ENABLE; removed none
- note added: "ENCODER QUADRATURE"
- note added: "UNUSED PICO PINS"
- moved on the sheet: C4, J5, J6, R8

Commit message: driver updates
Parts:
- added C10, C9: 10uF, symbol Device:C
- added U8: LM1117IMPX-5.0_NOPB, LM1117IMPX-5.0_NOPB:SOT230P700X180-4N, symbol LM1117IMPX-5.0_NOPB:LM1117IMPX-5.0_NOPB
- J5: symbol Connector:Screw_Terminal_01x03 -> Connector:Screw_Terminal_01x02
- R8: value R -> 5k; PART_NO (none) -> 1879246-3
- SW1: PART_NO (none) -> STO-060A24AB
Connections:
- net +12V: now also C9.1, U8.4 (VOUT)
- net +5V: now also C10.1, U8.2 (VOUT), U8.4 (VOUT); no longer J5.2 (Pin_2)
- net GND: now also J5.2 (Pin_2), C10.2, C9.2, U8.1 (GND); no longer J5.3 (Pin_3)
- net RP_CAN_INTERRUPT: now also U1.5 (GP3)
- net UNUSED_GP3: no longer U1.5 (GP3)
Other:
- sheet Analog ports: added none; removed A-IN_EXTRA_0, A-IN_EXTRA_1, A-IN_EXTRA_2, A-IN_EXTRA_3
- moved on the sheet: SW1
