File: Closed Loop Motor Driver CCA/Closed Loop Motor Driver/untitled.kicad_sch (KiCad schematic)
At the start: 5 parts, among them U2 DRV8871DDAR

Commit message: driver updates
Changed lines of the file:
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@@
   (junction (at 198.12 77.47) (diameter 0) (color 0 0 0 0)
   )
-  (junction (at 182.88 100.33) (diameter 0) (color 0 0 0 0)
-  )
-  (junction (at 182.88 97.79) (diameter 0) (color 0 0 0 0)
+  (junction (at 187.325 100.33) (diameter 0) (color 0 0 0 0)
+  )
+  (junction (at 187.325 97.79) (diameter 0) (color 0 0 0 0)
   )
   (junction (at 218.44 77.47) (diameter 0) (color 0 0 0 0)
@@
     (stroke (width 0) (type default))
   )
-  (wire (pts (xy 162.56 80.01) (xy 182.88 80.01))
+  (wire (pts (xy 169.545 85.09) (xy 162.56 85.09))
+    (stroke (width 0) (type default))
+  )
+  (wire (pts (xy 162.56 80.01) (xy 187.325 80.01))
+    (stroke (width 0) (type default))
+  )
+  (wire (pts (xy 169.545 87.63) (xy 162.56 87.63))
     (stroke (width 0) (type default))
   )
@@
     (stroke (width 0) (type default))
   )
-  (wire (pts (xy 162.56 100.33) (xy 182.88 100.33))
-    (stroke (width 0) (type default))
-  )
-  (wire (pts (xy 182.88 100.33) (xy 182.88 104.14))
-    (stroke (width 0) (type default))
-  )
-  (wire (pts (xy 162.56 97.79) (xy 182.88 97.79))
+  (wire (pts (xy 162.56 100.33) (xy 187.325 100.33))
+    (stroke (width 0) (type default))
+  )
+  (wire (pts (xy 187.325 100.33) (xy 187.325 104.14))
+    (stroke (width 0) (type default))
+  )
+  (wire (pts (xy 162.56 97.79) (xy 187.325 97.79))
     (stroke (width 0) (type default))
   )
@@
     (stroke (width 0) (type default))
   )
-  (wire (pts (xy 182.88 97.79) (xy 182.88 100.33))
-    (stroke (width 0) (type default))
-  )
-  (wire (pts (xy 182.88 80.01) (xy 182.88 97.79))
+  (wire (pts (xy 187.325 97.79) (xy 187.325 100.33))
+    (stroke (width 0) (type default))
+  )
+  (wire (pts (xy 187.325 80.01) (xy 187.325 97.79))
     (stroke (width 0) (type default))
   )
@@
     (stroke (width 0) (type default))
   )
-  (hierarchical_label "MOTOR_OUT2" (shape output) (at 162.56 87.63 0) (fields_autoplaced)
+  (hierarchical_label "MOTOR_OUT2" (shape output) (at 169.545 87.63 0) (fields_autoplaced)
     (effects (font (size 1.27 1.27)) (justify left))
   )
@@
     (effects (font (size 1.27 1.27)) (justify right))
   )
-  (hierarchical_label "MOTOR_OUT1" (shape output) (at 162.56 85.09 0) (fields_autoplaced)
+  (hierarchical_label "MOTOR_OUT1" (shape output) (at 169.545 85.09 0) (fields_autoplaced)
     (effects (font (size 1.27 1.27)) (justify left))
   )
   (hierarchical_label "MOTOR_IN1" (shape input) (at 127 87.63 180) (fields_autoplaced)
     (effects (font (size 1.27 1.27)) (justify right))
+  )
+  (netclass_flag "" (length 2.54) (shape round) (at 165.1 85.09 0) (fields_autoplaced)
+    (effects (font (size 1.27 1.27)) (justify left bottom))
+    (property "Netclass" "MOTOR_OUT" (at 165.7985 82.55 0)
+      (effects (font (size 1.27 1.27) italic) (justify left) hide)
+    )
   )
   (symbol (lib_id "DRV8871DDAR:DRV8871DDAR") (at 144.78 90.17 0) (unit 1)
@@
     )
   )
-  (symbol (lib_id "power:GND") (at 182.88 104.14 0) (unit 1)
-    (in_bom yes) (on_board yes) (dnp no) (fields_autoplaced)
-    (property "Reference" "#PWR01" (at 182.88 110.49 0)
-      (effects (font (size 1.27 1.27)) hide)
-    )
-    (property "Value" "GND" (at 182.88 109.22 0)
-      (effects (font (size 1.27 1.27)))
-    )
-    (property "Footprint" "" (at 182.88 104.14 0)
-      (effects (font (size 1.27 1.27)) hide)
-    )
-    (property "Datasheet" "" (at 182.88 104.14 0)
-      (effects (font (size 1.27 1.27)) hide)
-    )
+  (symbol (lib_id "power:GND") (at 187.325 104.14 0) (unit 1)
+    (in_bom yes) (on_board yes) (dnp no) (fields_autoplaced)
+    (property "Reference" "#PWR01" (at 187.325 110.49 0)
+      (effects (font (size 1.27 1.27)) hide)
+    )
+    (property "Value" "GND" (at 187.325 109.22 0)
+      (effects (font (size 1.27 1.27)))
+    )
+    (property "Footprint" "" (at 187.325 104.14 0)
+      (effects (font (size 1.27 1.27)) hide)
+    )
+    (property "Datasheet" "" (at 187.325 104.14 0)
+      (effects (font (size 1.27 1.27)) hide)
+    )
